File: hardware/initial-driver/power_handling.kicad_sch (KiCad schematic)
At the start: 31 parts, among them U2 TPS54260, U3 TPS54260

Commit message: add more stuff
Connections:
- net +3V3: now also C10.1, C11.1
- net Vdrive: no longer C10.1, C11.1
Other:
- moved on the sheet: C10, C11
