File: r-version/animated-robot.kicad_sch (KiCad schematic)
At the start: 86 parts, among them J1 USB_C_Receptacle_USB2.0_16P, J2 Conn_02x03_Odd_Even, J3 Conn_01x02, J4 Conn_01x05, J5 Conn_01x01, J6 Conn_01x01, J7 Conn_01x01, Q1 Q_NMOS_GDS, Q2 Q_NMOS_GDS, Q3 Q_NMOS_GDS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

Commit message: settle on a h-bridge design
Parts:
- removed D2, D5, D8: D_Small, symbol Device:D_Small
- added C19, C20, C21: C_Small, symbol Device:C_Small
- added D2, D5, D8: SS34, symbol Device:D_Schottky_Small
- C10, C14, C6: value C_Small -> 10 uF; LCSC (none) -> C13585
- C12, C16, C7: value C_Small -> 0.47 uF; LCSC (none) -> C13967
- D10, D3, D4, D6, D7, D9: value D_Small -> ES2JF; LCSC (none) -> C7420342
- Q1, Q2, Q3, Q4, Q5, Q6: value Q_NMOS_GDS -> WSD4070DN; LCSC (none) -> C719095
- R10, R15, R18, R20, R24, R26: value R_Small -> 10
- R14, R16, R19, R21, R25, R27: value R_Small -> 51
- R29, R31, R33, R35: value R_Small -> 56k
- R30, R32, R34, R36: value R_Small -> 10k
Connections:
- net +BATT: now also D2.2 (A), D5.2 (A), D8.2 (A)
- net BEMF0: now also C19.1
- net BEMF1: now also C20.1
- net BEMF2: now also C21.1
- net GND: now also C19.2, C20.2, C21.2
- net at R9.1: now also D2.1 (K)
- net at R23.1: now also D8.1 (K)
- net at R17.1: now also D5.1 (K)
Other:
- note added: "xxx not sure how to calculate optimal vals here"
- note added: "xxx ti says schottky is better?"
- note added: "xxx why is the devboard caps so big? https://www.ti.com/lit/an/slua887a/slua887a.pdf 0.1 uF > 10*Cg CL21B474KBFNNN derate -40% @ 20 V --> still > 0.2 uF"
