File: hardware/linkodrive08/linkodrive08.kicad_sch (KiCad schematic)
At the start: 145 parts, among them J1 USB_C_Receptacle_USB2.0_16P, J10 WCH_GPIO, J11 ENC, J12 LKS_SPI, J13 LKS_I2C, J14 WCH_UART_ALT, J15 LKS_SIF, J16 LKS_IO, J2 HALL, J3 WCH_SWD, J4 LKS_SWD, J5 MOT_POWER, J6 GATE_DRIVE, J7 LOGIC_POWER, J8 MOT, J9 CAN, Q1 WSD4070DN, Q2 WSD4070DN, Q3 WSD4070DN, Q4 WSD4070DN, Q5 WSD4070DN, Q6 WSD4070DN, U1 LKS32MC086NxQx, U2 CH32V203G6U6, U3 XL1509-ADJ, U4 SN65HVD230, U5 LGS5145, Y1 Crystal_GND24_Small

Commit message: Initial PCB work
Parts:
- added C37: 1n, Capacitor_SMD:C_0603_1608Metric, symbol Device:C_Small
- J10: footprint (none) -> Connector_PinSocket_2.54mm:PinSocket_2x05_P2.54mm_Vertical
- J11, J16, J2: footprint (none) -> Connector_PinSocket_2.54mm:PinSocket_1x05_P2.54mm_Vertical
- J12: footprint (none) -> Connector_PinSocket_2.54mm:PinSocket_1x06_P2.54mm_Vertical
- J13, J14: footprint (none) -> Connector_PinSocket_2.54mm:PinSocket_1x04_P2.54mm_Vertical
- J15, J8: footprint (none) -> Connector_PinSocket_2.54mm:PinSocket_1x03_P2.54mm_Vertical
- J5, J6, J7, J9: footprint (none) -> Connector_PinSocket_2.54mm:PinSocket_1x02_P2.54mm_Vertical
- L2: footprint (none) -> Inductor_SMD:L_Changjiang_FNR5040S; LCSC C13585 -> C167967
- Q1, Q2, Q3, Q4, Q5, Q6: value WSD4070DN -> HSU6066; footprint (none) -> Package_TO_SOT_SMD:TO-252-2; LCSC C719095 -> C22359249
- R1, R2: footprint (none) -> Resistor_SMD:R_0603_1608Metric; LCSC (none) -> C23186
- R11, R18, R26: footprint (none) -> Resistor_SMD:R_0603_1608Metric; LCSC (none) -> C23153
- R12, R20, R28, R44, R45: footprint (none) -> Resistor_SMD:R_0603_1608Metric; LCSC (none) -> C21190
- R30: footprint (none) -> Resistor_SMD:R_0603_1608Metric; LCSC (none) -> C4216
- R31: footprint (none) -> Resistor_SMD:R_0603_1608Metric; LCSC (none) -> C4184
- R32, R35, R36, R37, R39, R40: footprint (none) -> Resistor_SMD:R_0603_1608Metric
- R33: footprint (none) -> Resistor_SMD:R_0603_1608Metric; LCSC (none) -> C25808
- R41: value 500k -> 39k; footprint (none) -> Resistor_SMD:R_0603_1608Metric; LCSC (none) -> C23153
- R42: value 10k -> 1k; LCSC C25804 -> C21190
- R43: footprint (none) -> Resistor_SMD:R_0603_1608Metric; LCSC (none) -> C25803
Connections:
- net GND: now also C37.2
- net VBATT_MEAS: now also C37.1
Other:
- note added: "General notes"
- note added: "Possible other transistor options: - HSU6066 - C22359249 - WSD4070DN - C719095"
- note added: "Spec'd for ~160kHz cutoff"
- note added: "This is a dev board and is both subject to change and may not work"
- note added: "To spec the divder low pass filters: Calc thevamin resistance which in this simple case is te two resistors paralleled And then punch that value into your low pass filter calc"
