File: hardware/linkodrive08/linkodrive08.kicad_pcb (KiCad board)
At the start: 4 copper layers, 67.2 x 90.4 mm, 161 parts, among them J1 VBUS, J10 ENC, J11 LKS_I2C, J12 LKS_SWD, J13 HALL, J14 MOT_U, J15 MOT_V, J16 MOT_W, J17 WCH_GPIO, J18 WCH_UART_ALT, J19 GND, J2 USB_C_Receptacle_USB2.0_16P, J3 GATE_DRIVE, J4 LOGIC_POWER, J5 LKS_SIF, J6 LKS_IO, J7 LKS_SPI, J8 CAN, J9 WCH_SWD, Q1 JMTK80N06A, Q2 JMTK80N06A, Q3 JMTK80N06A, Q4 JMTK80N06A, Q5 JMTK80N06A, Q6 JMTK80N06A, U1 LKS32MC086NxQx, U2 SN65HVD230, U3 CH32V203G6U6, U4 XL1509-ADJ, U5 LGS5145, Y1 Crystal_GND24_Small

Commit message: changes?
Routing:
- net +3V3: track 177.2 -> 179.5 mm
- net /SPI_DI: track 45.5 -> 44.4 mm
- net /HALL_W: track 43.6 -> 44.5 mm
- net /LKS_SWDIO: track 28.1 -> 28.8 mm
- net /ENC_A: track 33.2 -> 32.5 mm
- net /WCH_~{RST}: track 24.5 -> 25.0 mm
- net /UART_ALT_TX: track 34.4 -> 33.9 mm
- net /MOT3: vias 340 -> 346
- net /MOT2: vias 340 -> 346
- net /MOT1: vias 340 -> 349
